File: BMS.kicad_sch (KiCad schematic)
At the start: 85 parts, among them IC1 BQ7695201PFBR, IC2 PMV213SN,215, IC3 PMV213SN,215, J1 Conn_01x04_Socket, J2 Conn_01x06_Pin, J3 Conn_01x02_Pin, J4 Conn_01x04_Socket, Q1 FCX495TA, Q2 NTMFS5C628NLT1G, Q3 NTMFS5C628NLT1G

Commit message: updated the schematic and uploaded the pcb file
Parts:
- removed C11, C21: 220nF, symbol Device:C_45deg
- removed D2, D3, D4, D5: D_Zener, symbol Device:D_Zener
- removed J1, J4: Conn_01x04_Socket, symbol Connector:Conn_01x04_Socket
- removed J2: Conn_01x06_Pin, symbol Connector:Conn_01x06_Pin
- removed R5, R6: 10k, symbol Device:R
- added J1: Conn_01x04_Pin, Connector_JST:JST_EH_B4B-EH-A_1x04_P2.50mm_Vertical, symbol Connector:Conn_01x04_Pin
- added J2: Conn_01x07_Pin, Connector_JST:JST_XH_B7B-XH-A_1x07_P2.50mm_Vertical, symbol Connector:Conn_01x07_Pin
- added J5: Conn_01x02_Pin, Connector_AMASS:AMASS_XT60-M_1x02_P7.20mm_Vertical, symbol Connector:Conn_01x02_Pin
- added R34, R35: 20, Resistor_SMD:R_0603_1608Metric_Pad0.98x0.95mm_HandSolder, symbol Device:R
- added TP1: BAT+, TestPoint:TestPoint_Pad_D1.0mm, symbol Connector:TestPoint
- added TP10, TP11, TP12, TP13, TP14, TP17, TP3, TP4, TP5: ~, TestPoint:TestPoint_Pad_D1.0mm, symbol Connector:TestPoint
- added TP15: PACK, TestPoint:TestPoint_Pad_D1.0mm, symbol Connector:TestPoint
- added TP16: LD, TestPoint:TestPoint_Pad_D1.0mm, symbol Connector:TestPoint
- added TP2: BAT, TestPoint:TestPoint_Pad_D1.0mm, symbol Connector:TestPoint
- added TP6: BAT-, TestPoint:TestPoint_Pad_D1.0mm, symbol Connector:TestPoint
- added TP7: SRP, TestPoint:TestPoint_Pad_D1.0mm, symbol Connector:TestPoint
- added TP8: SRN, TestPoint:TestPoint_Pad_D1.0mm, symbol Connector:TestPoint
- added TP9: TS2, TestPoint:TestPoint_Pad_D1.0mm, symbol Connector:TestPoint
- C1, C10, C12, C13, C14, C15, C16, C17, C18, C19, C2, C20, C22, C23, C24, C25, C26, C3, C4, C5, C6, C7, C8, C9: footprint (none) -> Capacitor_SMD:C_0603_1608Metric_Pad1.08x0.95mm_HandSolder
- D1, D11, D12, D6: footprint (none) -> V5N3M153M3I:V5N3M153M3I
- D10, D13, D8, D9: footprint (none) -> Diode_SMD:D_SOD-123
- D7: footprint (none) -> LED_SMD:LED_0603_1608Metric_Pad1.05x0.95mm_HandSolder
- IC1: footprint QFP50P900X900X120-48N -> BQ76952:QFP50P900X900X120-48N
- IC2, IC3: footprint SOT95P230X110-3N -> PMV213SN,215:SOT95P230X110-3N
- J3: footprint (none) -> Connector_PinHeader_2.54mm:PinHeader_1x02_P2.54mm_Vertical_SMD_Pin1Left
- NT1: footprint (none) -> NetTie:NetTie-2_SMD_Pad2.0mm
- Q1: footprint FCX495QTA -> FCX495TA:FCX495QTA
- Q2, Q3: footprint NTMFS5C628NLT1G:TRANS_NTMFS5C628NLT1G -> NTMFS5C628NLT1G:NTMFS5C460NLT1G
- R1, R10, R11, R12, R13, R14, R15, R16, R17, R18, R19, R2, R20, R21, R22, R23, R24, R25, R26, R27, R28, R29, R3, R30, R31, R32, R33, R4, R7, R8, R9, TH1, TH3: footprint (none) -> Resistor_SMD:R_0603_1608Metric_Pad0.98x0.95mm_HandSolder
Connections:
- net 6P: now also R15.1, J2.1 (Pin_1), TP1.1
- net BAT-: now also J2.7 (Pin_7), TP5.1, TP6.1
- net CHG: now also TP11.1
- net DSG: now also D11.5 (K), TP17.1; no longer D11.1 (K)
- net LD: now also TP16.1
- net PACK: now also TP15.1
- net PGND: now also C26.2, J1.2 (Pin_2), J5.1 (Pin_1)
- net at C10.2, IC1.1 (VC15): now also C12.1, IC1.2 (VC14), R11.2
- net at IC1.16 (VC0), R12.2: now also C20.2, IC1.15 (VC1)
- net at D9.1 (K), Q2.4, R20.2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: now also TP12.1
- net at C24.2, C25.1, D10.2 (A)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: now also J5.2 (Pin_2), TP13.1
- net at D10.1 (K), IC3.3 (D), R22.2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: now also TP14.1
- net at C5.1, C6.1, IC1.18 (SRP)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: now also TP7.1
- net at C17.2, C18.1, IC1.11 (VC5): now also IC1.10 (VC6), R34.2
- net at C18.2, IC1.12 (VC4): now also C19.1; no longer R13.2
- net at IC1.13 (VC3): now also C19.2, C20.1, IC1.14 (VC2), R35.2; no longer C19.1
- net at C5.2, C6.2, IC1.20 (SRN)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: now also TP8.1
- net at IC1.21 (TS1), TH1.1: now also TP4.1
- net at IC1.22 (TS2), J3.2 (Pin_2): now also TP9.1
- net at IC1.23 (TS3), TH3.1: now also TP10.1
- net at IC1.26 (SCL): now also J1.1 (Pin_1)
- net at IC1.27 (SDA): now also J1.3 (Pin_3)
- net at C12.2, IC1.3 (VC13): now also C13.1; no longer IC1.4 (VC12), R11.2
- net at C7.2, IC1.46 (CP1): now also TP3.1
- net at C7.1, C8.1, C9.1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: now also TP2.1
- net at IC1.5 (VC11): now also C13.2, C14.1, IC1.4 (VC12), R13.2; no longer C13.1
- net at C14.2, C15.1: now also IC1.6 (VC10); no longer IC1.7 (VC9)
- net at C15.2, IC1.8 (VC8), R14.2: now also C16.1, IC1.7 (VC9)
- net at C16.2, IC1.9 (VC7): now also C17.1
- net at R11.1: now also J2.2 (Pin_2)
- net at R14.1: now also J2.4 (Pin_4)
- net at R13.1: now also J2.3 (Pin_3)
- net at R2.1: now also D1.5 (K); no longer D1.1 (K)
- net at R28.2: now also D12.5 (K); no longer D12.1 (K)
- net at R10.1: now also D6.5 (K); no longer D6.1 (K)
- net REG1: no longer names the net of C3.1, IC1.35 (REG1)
- net VSS renamed GND
- new net: J2.5 (Pin_5), R34.1
- new net: J2.6 (Pin_6), R35.1
- no-connect marks 7 -> 8
Other:
- note added: "PACK+ PACK-"
- note removed: "PACK+ PACK+ PACK- PACK-"
- moved on the sheet: C10, C12, D12, R11
